File: Hardware/DCMotorDriver/DCMotorDriver.kicad_pcb (KiCad board)
At the start: 2 copper layers, 69 parts, among them J1 J-Tag, J10 01x02 JST, J2 Screw_Terminal_01x02, J3 USB_C_Receptacle_USB2.0, J4 01x02 JST, J5 01x04 JST, J6 01x02 JST, J7 Screw_Terminal_01x02, J8 01x02 JST, J9 01x02 JST, Q1 PMOS, Q2 NMOS, Q3 NMOS, SW1 SW_Push, SW2 SW_Push, U1 STM32F401CCUx, U2 DRV8848, U3 TPS62133, U4 AZ1117-3.3, Y1 25Mhz

Commit message: update
Parts:
- removed C1, C20: 1u, Capacitor_SMD:C_0402_1005Metric
- removed C10: 4u7, Capacitor_SMD:C_0402_1005Metric
- removed C11, C12, C13, C24: 2u2, Capacitor_SMD:C_0402_1005Metric
- removed C14, C15: 12p, Capacitor_SMD:C_0402_1005Metric
- removed C16, C2, C23, C25, C4, C5, C6, C7, C8: 100n, Capacitor_SMD:C_0402_1005Metric
- removed C17, C21, C9: 10u, Capacitor_SMD:C_0402_1005Metric
- removed C18, C22: 22u, Capacitor_SMD:C_0402_1005Metric
- removed C19: 3n3, Capacitor_SMD:C_0402_1005Metric
- removed C3: 220u, Capacitor_SMD:C_0402_1005Metric
- removed D1: 2 A, Diode_SMD:D_0603_1608Metric
- removed D2: 5V1, Diode_SMD:D_0402_1005Metric
- removed D3: LED, Diode_SMD:D_0402_1005Metric
- removed FB1, FB2: 220R @100Mhz, Inductor_SMD:L_0402_1005Metric
- removed J1: J-Tag, Connector:Tag-Connect_TC2030-IDC-FP_2x03_P1.27mm_Vertical
- removed J10, J4, J6, J8, J9: 01x02 JST, Connector_JST:JST_EH_B2B-EH-A_1x02_P2.50mm_Vertical
- removed J2, J7: Screw_Terminal_01x02, Connector_PinHeader_2.54mm:PinHeader_1x02_P2.54mm_Horizontal
- removed J3: USB_C_Receptacle_USB2.0, Connector_USB:USB_C_Receptacle_XKB_U262-16XN-4BVC11
- removed J5: 01x04 JST, Connector_JST:JST_EH_B4B-EH-A_1x04_P2.50mm_Vertical
- removed L1: 2u2, Inductor_SMD:L_0805_2012Metric
- removed Q1: PMOS, Package_TO_SOT_SMD:SOT-23-3
- removed Q2, Q3: NMOS, Package_TO_SOT_SMD:SOT-23-3
- removed R1, R10, R11, R7: 10k, Resistor_SMD:R_0402_1005Metric
- removed R12: 100k, Resistor_SMD:R_0402_1005Metric
- removed R13, R8: 0R, Resistor_SMD:R_0402_1005Metric
- removed R14, R15: 1k2, Resistor_SMD:R_0402_1005Metric
- removed R2, R3: 2k2, Resistor_SMD:R_0402_1005Metric
- removed R4: 1M, Resistor_SMD:R_0402_1005Metric
- removed R5, R6: 5k1, Resistor_SMD:R_0402_1005Metric
- removed R9: 1k, Resistor_SMD:R_0402_1005Metric
- removed SW1, SW2: SW_Push, Button_Switch_SMD:SW_Push_1P1T_NO_CK_KMR2
- removed TP1, TP2, TP3: TestPoint, TestPoint:TestPoint_Pad_D1.0mm
- removed U1: STM32F401CCUx, Package_DFN_QFN:QFN-48-1EP_7x7mm_P0.5mm_EP5.6x5.6mm
- removed U2: DRV8848, Package_SO:TSSOP-16-1EP_4.4x5mm_P0.65mm
- removed U3: TPS62133, Package_DFN_QFN:VQFN-16-1EP_3x3mm_P0.5mm_EP1.68x1.68mm_ThermalVias
- removed U4: AZ1117-3.3, Package_TO_SOT_SMD:SOT-223-3_TabPin2
- removed Y1: 25Mhz, Crystal:Crystal_SMD_0603-4Pin_6.0x3.5mm
