File: Hardware/DCMotorDriver/DCMotorDriver.kicad_sch (KiCad schematic)
At the start: 74 parts, among them J1 J-Tag, J10 01x02 JST, J11 01x02 JST, J12 01x02 JST, J13 01x02 JST, J14 01x02 JST, J15 01x02 JST, J2 Screw_Terminal_01x02, J3 USB_C_Receptacle_USB2.0, J4 01x02 JST, J5 01x04 JST, J6 01x02 JST, J7 Screw_Terminal_01x02, J8 01x02 JST, J9 01x02 JST, Q1 PMOS, Q2 NMOS, Q3 NMOS, SW1 SW_Push, SW2 SW_Push, U1 STM32F401CCUx, U2 DRV8848, U3 TPS62133, U4 AZ1117-3.3, Y1 25Mhz

Commit message: layout v1
Parts:
- removed J11, J12, J13, J14, J15: 01x02 JST, Connector_JST:JST_EH_B2B-EH-A_1x02_P2.50mm_Vertical, symbol Connector:Conn_01x02_Socket
- removed TP4: TestPoint, symbol Connector:TestPoint
- added C25: 100n, Capacitor_SMD:C_0402_1005Metric, symbol Device:C_Small
- C1, C10, C11, C12, C13, C14, C15, C16, C17, C18, C19, C2, C20, C21, C22, C23, C24, C3, C4, C5, C6, C7, C8, C9: footprint (none) -> Capacitor_SMD:C_0402_1005Metric
- D1: footprint (none) -> Diode_SMD:D_0603_1608Metric
- D2, D3: footprint (none) -> Diode_SMD:D_0402_1005Metric
- FB1, FB2: footprint (none) -> Inductor_SMD:L_0402_1005Metric
- J2, J7: footprint (none) -> Connector_PinHeader_2.54mm:PinHeader_1x02_P2.54mm_Horizontal
- L1: footprint (none) -> Inductor_SMD:L_0805_2012Metric
- Q1, Q2, Q3: footprint (none) -> Package_TO_SOT_SMD:SOT-23-3
- R1, R10, R11, R12, R13, R14, R15, R2, R3, R4, R5, R6, R7, R8, R9: footprint (none) -> Resistor_SMD:R_0402_1005Metric
- SW1, SW2: footprint (none) -> Button_Switch_SMD:SW_Push_1P1T_NO_CK_KMR2
- TP1, TP2, TP3: footprint (none) -> TestPoint:TestPoint_Pad_D1.0mm
- Y1: footprint (none) -> Crystal:Crystal_SMD_0603-4Pin_6.0x3.5mm
Connections:
- net SCL is gone; now on net I2C1_SCL: Q2.3 (S), R15.2
- net SDA is gone; now on net I2C1_SDA: Q3.3 (S), R14.2
- net SWIDO is gone; now on net SWDIO: U1.34 (PA13)
- net +3V3: now also C25.1
- net GND: now also C25.2
Other:
- company: (none) -> WROBOTICS
- title: (none) -> DC Motor Controller
- moved on the sheet: C6, C7, C8

Commit message: update
Parts:
- removed C24: 2u2, Capacitor_SMD:C_0402_1005Metric, symbol Device:C_Small
- removed D2: 5V1, Diode_SMD:D_0402_1005Metric, symbol Device:D_Zener
- removed TP3: TestPoint, TestPoint:TestPoint_Pad_D1.0mm, symbol Connector:TestPoint
- added C23: 2u2, Capacitor_SMD:C_0402_1005Metric, symbol Device:C_Small
- added D1: 12v6, Diode_SMD:D_0402_1005Metric, symbol Device:D_Zener
- added D2: D_Schottky, Diode_SMD:D_0402_1005Metric, symbol Device:D_Schottky
- added D4: BAT54, Diode_SMD:D_1210_3225Metric, symbol Device:D_Schottky
- added J1: Screw_Terminal_01x02, TerminalBlock_4Ucon:TerminalBlock_4Ucon_1x02_P3.50mm_Vertical, symbol Connector:Screw_Terminal_01x02
- added J2, J4, J6: 01x02 JST, Connector_JST:JST_EH_B2B-EH-A_1x02_P2.50mm_Vertical, symbol Connector:Conn_01x02_Socket
- added Q2: PMOS, Package_TO_SOT_SMD:SOT-723, symbol Simulation_SPICE:PMOS
- added Q3: PMOS, Package_TO_SOT_SMD:SOT-23-3, symbol Simulation_SPICE:PMOS
- added Q4: NMOS, Package_TO_SOT_SMD:SOT-723, symbol Simulation_SPICE:NMOS
- added R1: 0R, Resistor_SMD:R_0402_1005Metric, symbol Device:R_Small
- added R10, R4: 100k, Resistor_SMD:R_0402_1005Metric, symbol Device:R_Small
- added R11, R7: 10k, Resistor_SMD:R_0402_1005Metric, symbol Device:R_Small
- added R2, R3: 5k1, Resistor_SMD:R_0402_1005Metric, symbol Device:R_Small
- added U2: USBLC6-2SC6, Package_TO_SOT_SMD:SOT-23-6, symbol Power_Protection:USBLC6-2SC6
- added U3: AMS1117-3.3, Package_TO_SOT_SMD:SOT-223-3_TabPin2, symbol Regulator_Linear:AMS1117-3.3
- C1: renamed from C21; footprint Capacitor_SMD:C_0402_1005Metric -> Capacitor_SMD:C_0603_1608Metric
- C10: footprint Capacitor_SMD:C_0402_1005Metric -> Capacitor_SMD:C_0603_1608Metric
- C11: renamed from C9; footprint Capacitor_SMD:C_0402_1005Metric -> Capacitor_SMD:C_0603_1608Metric
- C17: renamed from C3; footprint Capacitor_SMD:C_0402_1005Metric -> Capacitor_SMD:C_1206_3216Metric
- C6: renamed from C22; footprint Capacitor_SMD:C_0402_1005Metric -> Capacitor_SMD:C_0603_1608Metric
- C8: renamed from C17; footprint Capacitor_SMD:C_0402_1005Metric -> Capacitor_SMD:C_0603_1608Metric
- C9: renamed from C18; footprint Capacitor_SMD:C_0402_1005Metric -> Capacitor_SMD:C_0603_1608Metric
- J11: renamed from J7; footprint Connector_PinHeader_2.54mm:PinHeader_1x02_P2.54mm_Horizontal -> TerminalBlock_4Ucon:TerminalBlock_4Ucon_1x02_P3.50mm_Vertical
- J13: renamed from J2; footprint Connector_PinHeader_2.54mm:PinHeader_1x02_P2.54mm_Horizontal -> TerminalBlock_4Ucon:TerminalBlock_4Ucon_1x02_P3.50mm_Vertical
- Q5: renamed from Q2; footprint Package_TO_SOT_SMD:SOT-23-3 -> Package_TO_SOT_SMD:SOT-723
- Q6: renamed from Q3; footprint Package_TO_SOT_SMD:SOT-23-3 -> Package_TO_SOT_SMD:SOT-723
- R6: value 5k1 -> 200k
- R8: value 0R -> 1M
- SW1, SW2: footprint Button_Switch_SMD:SW_Push_1P1T_NO_CK_KMR2 -> Button_Switch_THT:SW_PUSH_6mm
- renumbered C25 to C12, C8 to C13, C7 to C14, C6 to C15, C2 to C16, C15 to C18, C14 to C19, C20 to C2, C1 to C21, C4 to C22, C5 to C24, C16 to C25, C13 to C26, C12 to C3, C11 to C4, C23 to C5, C19 to C7, J6 to J10, J5 to J12, J1 to J14, J10 to J3, J3 to J5, J8 to J7, J9 to J8, J4 to J9, R1 to R12, R9 to R13, R15 to R14, R14 to R15, R11 to R16, R10 to R17, R12 to R5, R4 to R9, U3 to U1, U2 to U4, U1 to U5
Connections:
- net +3.3V: now also C23.1, U3.2 (VO); no longer J14.1 (VCC), Q5.2 (G), U4.2 (VO)
- net +3V3: no longer C12.1
- net +5V: now also Q3.1 (D); no longer Q1.3 (S)
- net +BATT: now also D1.1 (K), Q2.3 (S), R1.1, R7.1; no longer C2.1, R13.1
- net AIN_2: no longer U4.15 (AIN2)
- net DRV_Fault: no longer U5.15 (PA5)
- net ENC1_B: no longer J7.2 (Pin_2)
- net GND: now also C23.2, Q4.3 (S), R10.2, R2.1, U3.1 (GND); no longer C12.2, C4.2, C8.2, J12.2 (Pin_2), R5.2, R6.2, R7.2, U1.6 (AGND), U4.1 (GND), U4.13 (GND), U4.17 (PPAD)
- net I2C1_SDA: no longer R3.2
- net SWDIO: no longer J14.2 (SWDIO)
- net USB2_N: now also U2.4 (I/O2); no longer J5.A7 (D-), J5.B7 (D-)
- net USB2_P: now also U2.3 (I/O2); no longer J5.A6 (D+), J5.B6 (D+)
- net VBUS: now also Q3.2 (G); no longer C3.1, D1.2 (A), FB1.2, Q1.2 (G), R7.1
- net VCC: now also Q3.3 (S), U3.3 (VI); no longer D1.1 (K), J12.1 (Pin_1), Q1.1 (D), U4.3 (VI)
- net XTAL_OUT: now also C19.1, Y1.3; no longer R8.2
- net at C5.1, L1.2, R5.1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: no longer FB2.1
- net at C22.2, U4.4 (AOUT2): no longer J11.2 (Pin_2)
- net at U1.1 (SW), U1.2 (SW), U1.3 (SW): no longer L1.1
- net at U1.13 (EN): now also R1.2; no longer R13.2
- net PA6: now reaches U5.16 (PA6)
- net PA6: now also J2.1 (Pin_1)
- net PA7: now reaches U5.17 (PA7)
- net PB10: now reaches U5.21 (PB10)
- net PB10: now also J3.2 (Pin_2)
- net PB12: now reaches U5.25 (PB12)
- net PB12: now also J4.1 (Pin_1)
- net PB13: now reaches U5.26 (PB13)
- net PB13: now also J4.2 (Pin_2)
- net PA8: now reaches U5.29 (PA8)
- net PA8: now also J3.1 (Pin_1)
- net PC14: now reaches U5.3 (PC14)
- net PC15: now reaches U5.4 (PC15)
- net at FB1.1, J5.A4 (VBUS), J5.A9 (VBUS)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: no longer C4.1
- net at J5.A5 (CC1): now also R3.2; no longer R5.1
- net at R6.1: now also Q2.1 (D); no longer J5.B5 (CC2)
- new net: Q2.2 (G), Q4.1 (D), R7.2
- new net: U4.13 (GND), U4.17 (PPAD)
- new net: D1.2 (A), R4.1
- new net: J5.A7 (D-), J5.B7 (D-), U2.6 (I/O1)
- new net: C3.1, FB1.2
- new net: J5.A6 (D+), J5.B6 (D+)
- new net BAT_MON: R6.2
- new net PB14: J6.1 (Pin_1)
- new net PB15: J6.2 (Pin_2)
- new net VBAT: J1.1 (Pin_1), Q1.1 (D)
- now unconnected: R8.1
- no-connect marks 14 -> 9
Other:
- note added: "Power Supply"
- note added: "USB 2.0 FS Type C"
- note removed: "12 GPIOs free"
- note removed: "Power Supply & USB C"
- moved on the sheet: C1, C11, C13, C14, C15, C16, C17, C18, C19, C2, C21, C22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
