File: Hardware/PiCardZW/PiCardZW.kicad_sch (KiCad schematic)
At the start: 3 parts

Commit message: desingDocs
Parts:
- added C1, C3: 10u, Capacitor_THT:CP_Radial_D4.0mm_P1.50mm, symbol Device:C_Polarized_Small_US
- added C2: 100u, Capacitor_THT:CP_Radial_D4.0mm_P1.50mm, symbol Device:C_Polarized_Small_US
- added H1, H2, H3, H4: MountingHole, MountingHole:MountingHole_3.2mm_M3, symbol Mechanical:MountingHole
- added J1, J12, J8: Screw_Terminal_01x02, Connector_JST:JST_EH_B2B-EH-A_1x02_P2.50mm_Vertical, symbol Connector:Screw_Terminal_01x02
- added J10, J9: Conn_01x08, Connector_PinSocket_2.54mm:PinSocket_1x08_P2.54mm_Vertical, symbol Connector_Generic:Conn_01x08
- added J11, J4, J5: Conn_01x04, Connector_JST:JST_EH_B4B-EH-A_1x04_P2.50mm_Vertical, symbol Connector_Generic:Conn_01x04
- added J3: Conn_01x02, Connector_JST:JST_EH_B2B-EH-A_1x02_P2.50mm_Vertical, symbol Connector_Generic:Conn_01x02
- J2: renamed from J?; footprint (none) -> Connector_PinSocket_2.54mm:PinSocket_2x20_P2.54mm_Vertical
- J6, J7: renamed from J?; footprint (none) -> Connector_PinSocket_2.54mm:PinSocket_1x20_P2.54mm_Vertical
Connections:
- net 5V_STM is gone; now on net +5V: J6.18 (Pin_18), J7.1 (Pin_1)
- net PA10 is gone; now on net DEBUG_RX: J6.7 (Pin_7)
- net PA9 is gone; now on net DEBUG_TX: J6.6 (Pin_6)
- net R is gone; now on net nRST: J7.16 (Pin_16)
- net GND: now also C1.2, C2.2, C3.2, J1.2 (Pin_2), J10.3 (Pin_3), J10.8 (Pin_8), J11.2 (Pin_2), J3.2 (Pin_2), J4.1 (Pin_1), J5.1 (Pin_1), J9.8 (Pin_8)
- net 3V3_Pi: no longer names the net of J2.1 (Pin_1)
- net 3V3_Pi: no longer J2.17 (Pin_17)
- net 3V3_STM renamed +3.3V
- net +3.3V: now also C3.1, J11.1 (Pin_1), J4.2 (Pin_2), J5.2 (Pin_2)
- net 5V_PI renamed +5V
- net +5V: now also C1.1, J3.1 (Pin_1)
- net GPIO0_ID_SD: no longer names the net of J2.27 (Pin_27)
- net GPIO10_MOSI: no longer names the net of J2.19 (Pin_19)
- net GPIO11_SCLK: no longer names the net of J2.23 (Pin_23)
- net GPIO12_PWM0: no longer names the net of J2.32 (Pin_32)
- net GPIO13_PWM1: no longer names the net of J2.33 (Pin_33)
- net GPIO14_TXD renamed DEBUG_RX
- net GPIO15_RXD renamed DEBUG_TX
- net GPIO16: no longer names the net of J2.36 (Pin_36)
- net GPIO17: no longer names the net of J2.11 (Pin_11)
- net GPIO18_PCM_CLK: no longer names the net of J2.12 (Pin_12)
- net GPIO19_PCM_FS: no longer names the net of J2.35 (Pin_35)
- net GPIO1_ID_SC: no longer names the net of J2.28 (Pin_28)
- net GPIO20_PCM_DIN: no longer names the net of J2.38 (Pin_38)
- net GPIO21_PCM_DOUT: no longer names the net of J2.40 (Pin_40)
- net GPIO22: no longer names the net of J2.15 (Pin_15)
- net GPIO23: no longer names the net of J2.16 (Pin_16)
- net GPIO24: no longer names the net of J2.18 (Pin_18)
- net GPIO25: no longer names the net of J2.22 (Pin_22)
- net GPIO26: no longer names the net of J2.37 (Pin_37)
- net GPIO27: no longer names the net of J2.13 (Pin_13)
- net GPIO2_SDA: no longer names the net of J2.3 (Pin_3)
- net GPIO3_SCL: no longer names the net of J2.5 (Pin_5)
- net GPIO4_GPCLK0: no longer names the net of J2.7 (Pin_7)
- net GPIO5 renamed nRST
- net GPIO6: no longer names the net of J2.31 (Pin_31)
- net GPIO7_CE1: no longer names the net of J2.26 (Pin_26)
- net GPIO8_CE9: no longer names the net of J2.24 (Pin_24)
- net GPIO9_MISO: no longer names the net of J2.21 (Pin_21)
- net PA0 renamed ML_PWMA
- net ML_PWMA: now also J9.2 (Pin_2)
- net PA1 renamed ML_PWMB
- net ML_PWMB: now also J9.3 (Pin_3)
- net PA11: no longer names the net of J6.8 (Pin_8)
- net PA12: no longer names the net of J6.9 (Pin_9)
- net PA15: no longer names the net of J6.10 (Pin_10)
- net PA2 renamed MR_PWMA
- net MR_PWMA: now also J9.5 (Pin_5)
- net PA3 renamed MR_PWMB
- net MR_PWMB: now also J9.6 (Pin_6)
- net PA4 renamed DRV_EN
- net DRV_EN: now also J9.4 (Pin_4)
- net PA5: no longer names the net of J7.10 (Pin_10)
- net PA6: no longer names the net of J7.9 (Pin_9)
- net PA7: no longer names the net of J7.8 (Pin_8)
- net PA8: no longer names the net of J6.5 (Pin_5)
- net PB1: no longer names the net of J7.6 (Pin_6)
- net PB10: no longer names the net of J7.4 (Pin_4)
- net PB10: no longer J7.7 (Pin_7)
- net PB12: no longer names the net of J6.1 (Pin_1)
- net PB13: no longer names the net of J6.2 (Pin_2)
- net PB14: no longer names the net of J6.3 (Pin_3)
- net PB15: no longer names the net of J6.4 (Pin_4)
- net PB2: no longer names the net of J7.5 (Pin_5)
- net PB3: no longer names the net of J6.11 (Pin_11)
- net PB4 renamed ENCL_A
- net ENCL_A: now also J4.4 (Pin_4)
- net PB5 renamed ENCL_B
- net ENCL_B: now also J4.3 (Pin_3)
- net PB6 renamed ENCR_A
- net ENCR_A: now also J5.4 (Pin_4)
- net PB7 renamed ENCR_B
- net ENCR_B: now also J5.3 (Pin_3)
- net PB8 renamed IMU_SCL
- net IMU_SCL: now also J11.3 (Pin_3)
- net PB9 renamed IMU_SDA
- net IMU_SDA: now also J11.4 (Pin_4)
- net PC13: no longer names the net of J7.19 (Pin_19)
- net PC14: no longer names the net of J7.18 (Pin_18)
- net PC15: no longer names the net of J7.17 (Pin_17)
- net VBAT: no longer names the net of J7.20 (Pin_20)
- new net AOUT1: J10.4 (Pin_4), J8.2 (Pin_2)
- new net AOUT2: J10.5 (Pin_5), J8.1 (Pin_1)
- new net BOUT1: J10.6 (Pin_6), J12.2 (Pin_2)
- new net BOUT2: J10.7 (Pin_7), J12.1 (Pin_1)
- new net VM: C2.1, J1.1 (Pin_1), J10.1 (Pin_1)
- no-connect marks 0 -> 50
Other:
- note added: "3V3_Pi"
- note added: "BOARD POWER"
- note added: "DRV8833"
- note added: "ENCODER"
- note added: "GPIO0_ID_SD"
- note added: "GPIO10_MOSI"
- note added: "GPIO11_SCLK"
- note added: "GPIO12_PWM0"
- note added: "GPIO13_PWM1"
- note added: "GPIO14_TXD"
- note added: "GPIO15_RXD"
- note added: "GPIO16"
- note added: "GPIO17"
- note added: "GPIO18_PCM_CLK"
- note added: "GPIO19_PCM_FS"
- note added: "GPIO1_ID_SC"
- note added: "GPIO20_PCM_DIN"
- note added: "GPIO21_PCM_DOUT"
- note added: "GPIO22"
- note added: "GPIO23"
- note added: "GPIO24"
- note added: "GPIO25"
- note added: "GPIO26"
- note added: "GPIO27"
- note added: "GPIO2_SDA"
- note added: "GPIO3_SCL"
- note added: "GPIO4_GPCLK0"
- note added: "GPIO5"
- note added: "GPIO6"
- note added: "GPIO7_CE1"
- note added: "GPIO8_CE9"
- note added: "GPIO9_MISO"
- note added: "IMU"
- note added: "MOTOR CONN"
- note added: "MOTOR POWER"
- note added: "PA0"
- note added: "PA1"
- note added: "PA10"
- note added: "PA11"
- note added: "PA12"
- note added: "PA15"
- note added: "PA2"
- note added: "PA3"
- note added: "PA4"
- note added: "PA5"
- note added: "PA6"
- note added: "PA7"
- note added: "PA8"
- note added: "PA9"
- note added: "PB1"
- note added: "PB10"
- note added: "PB12"
- note added: "PB13"
- note added: "PB14"
- note added: "PB15"
- note added: "PB2"
- note added: "PB3"
- note added: "PB4"
- note added: "PB5"
- note added: "PB6"
- note added: "PB7"
- note added: "PB8"
- note added: "PB9"
- note added: "PC13"
- note added: "PC14"
- note added: "PC15"
- note added: "PI ZeroW"
- note added: "R"
- note added: "STM32F401RE"
- note added: "VBAT"
- moved on the sheet: J2, J6, J7

Commit message: eod
Parts:
- removed J10, J9: Conn_01x08, Connector_PinSocket_2.54mm:PinSocket_1x08_P2.54mm_Vertical, symbol Connector_Generic:Conn_01x08
- removed J11: Conn_01x04, Connector_JST:JST_EH_B4B-EH-A_1x04_P2.50mm_Vertical, symbol Connector_Generic:Conn_01x04
- removed J6, J7: Conn_01x20, Connector_PinSocket_2.54mm:PinSocket_1x20_P2.54mm_Vertical, symbol Connector_Generic:Conn_01x20
- added C4: 22u, Capacitor_THT:CP_Radial_D4.0mm_P1.50mm, symbol Device:C_Polarized_Small_US
- added J10, J11, J14, J9: Conn_01x07, symbol Connector_Generic:Conn_01x07
- added J13: Conn_01x05, symbol Connector_Generic:Conn_01x05
- added R1, R2: 10k, symbol Device:R_Small
- added R3: 100k, symbol Device:R_Small
- added R4: 1M, symbol Device:R_Small
- added U1: STM32F401CBUx, Package_DFN_QFN:QFN-48-1EP_7x7mm_P0.5mm_EP5.6x5.6mm, symbol MCU_ST_STM32F4:STM32F401CBUx
- added U2, U3: DRV8872DDA, Package_SO:Texas_HTSOP-8-1EP_3.9x4.9mm_P1.27mm_EP2.95x4.9mm_Mask2.4x3.1mm_ThermalVias, symbol Driver_Motor:DRV8872DDA
- added U4, U5: DRV8874QPWPRQ1, PWP0016J_N, symbol Driver_Motor:DRV8874QPWPRQ1
- C2: value 100u -> 22u; Voltage (none) -> 50V
Connections:
- net +3.3V: now also J13.1 (Pin_1), R1.1, R2.1
- net AOUT1: now also J11.3 (Pin_3)
- net AOUT2: now also J11.4 (Pin_4)
- net BOUT1: now also J9.3 (Pin_3)
- net BOUT2: now also J9.4 (Pin_4)
- net DEBUG_RX: now also U1.33 (PA12); no longer J2.8 (Pin_8)
- net DEBUG_TX: now also U1.32 (PA11); no longer J2.10 (Pin_10)
- net DRV_EN: now also J10.5 (Pin_5), J10.6 (Pin_6), J14.5 (Pin_5), J14.6 (Pin_6), U1.10 (PA0)
- net ENCL_A: now also U1.40 (PB4)
- net ENCL_B: now also U1.41 (PB5)
- net ENCR_A: now also U1.42 (PB6)
- net ENCR_B: now also U1.43 (PB7)
- net GND: now also C4.2, J10.2 (Pin_2), J11.2 (Pin_2), J13.2 (Pin_2), J14.2 (Pin_2), J9.2 (Pin_2), R4.2
- net IMU_SCL: now also J13.3 (Pin_3), U1.45 (PB8)
- net IMU_SDA: now also J13.4 (Pin_4), U1.46 (PB9)
- net ML_PWMA: now also J14.3 (Pin_3), U1.14 (PA4)
- net ML_PWMB: now also J14.4 (Pin_4), U1.13 (PA3)
- net MR_PWMA: now also J10.3 (Pin_3), U1.12 (PA2)
- net MR_PWMB: now also J10.4 (Pin_4), U1.11 (PA1)
- net VM: now also C4.1, J11.1 (Pin_1), J9.1 (Pin_1), R3.1
- net nRST: now also U1.7 (NRST)
- new net: J11.6 (Pin_6), R1.2
- new net: U3.1 (GND), U3.9 (GND)
- new net: J9.6 (Pin_6), R2.2
- new net: U2.1 (GND), U2.9 (GND)
- new net: U1.23 (VSS), U1.35 (VSS), U1.47 (VSS), U1.49 (VSS)
- new net IMU_INT: J13.5 (Pin_5)
- new net ML_CS: J11.7 (Pin_7), U1.16 (PA6)
- new net MR_CS: J9.7 (Pin_7), U1.17 (PA7)
- new net SERIAL_RX: J2.8 (Pin_8), U1.31 (PA10)
- new net SERIAL_TX: J2.10 (Pin_10), U1.30 (PA9)
- new net SPI2_MISO: U1.27 (PB14)
- new net SPI2_MOSI: U1.28 (PB15)
- new net SPI2_NSS2: U1.29 (PA8)
- new net SPI2_SCK: U1.26 (PB13)
- new net V_SENSE_M: R3.2, R4.1
- no-connect marks 50 -> 41
Other:
- note added: "CS"
- note added: "DRV8874 H Bridge"
- note added: "GND"
- note added: "IMODE"
- note added: "IN1"
- note added: "IN2"
- note added: "N_FLT"
- note added: "N_SLP"
- note added: "OUT1"
- note added: "OUT2"
- note added: "PMODE"
- note added: "VIN"
- note added: "VM"
- note added: "VREF"
- note removed: "DRV8833"
- note removed: "PA15"
- note removed: "PB3"
- moved on the sheet: C3, J12, J2, J8
